Commit message: added new world file

File: src/nav2_bringup/urdf/autobot.urdf (robot description, URDF)
Before this commit: robot autobot, 6 links, 5 joints
Joints:
- joint castor_wheels_joint: type fixed -> revolute

Commit message: added changes from detetched commit

File: src/nav2_bringup/urdf/autobot.urdf (robot description, URDF)
Before this commit: robot autobot, 6 links, 5 joints
Joints:
- joint castor_wheels_joint: type revolute -> fixed
